Commit message: Physics working

File: description/urdf/properties.xacro (robot description, xacro)
@@ -15,4 +15,4 @@
   <xacro:property name="ROLLER_RADIUS" value="0.006233225"/>
   <xacro:property name="ROLLER_MASS" value="0.1"/>
-  <xacro:property name="WHEEL_SCALE" value="1.33297475178"/>
+  <xacro:property name="WHEEL_SCALE" value="1.33297475178"/> <!-- 1.33297475178 -->
 </robot>

File: description/urdf/robotino.urdf (robot description, URDF)
Before this commit: robot robotino, 35 links, 34 joints
Links:
- link chassis_link: geometry collision cylinder length=0.05 radius=0.18; visual mesh filename=package://robotino_roller/description/mesh/robotino_base.dae scale=0.01 0.01 0.01
- link roller_lefttdownback_wheel0_link: geometry collision mesh filename=package://robotino_roller/description/mesh/roller01.stl; visual mesh filename=package://robotino_roller/description/mesh/roller01.stl
- link roller_lefttdownback_wheel1_link: geometry collision mesh filename=package://robotino_roller/description/mesh/roller01.stl; visual mesh filename=package://robotino_roller/description/mesh/roller01.stl
- link roller_lefttdownback_wheel2_link: geometry collision mesh filename=package://robotino_roller/description/mesh/roller01.stl; visual mesh filename=package://robotino_roller/description/mesh/roller01.stl
- link roller_lefttdownfront_wheel0_link: geometry collision mesh filename=package://robotino_roller/description/mesh/roller01.stl; visual mesh filename=package://robotino_roller/description/mesh/roller01.stl
- link roller_lefttdownfront_wheel1_link: geometry collision mesh filename=package://robotino_roller/description/mesh/roller01.stl; visual mesh filename=package://robotino_roller/description/mesh/roller01.stl
- link roller_lefttdownfront_wheel2_link: geometry collision mesh filename=package://robotino_roller/description/mesh/roller01.stl; visual mesh filename=package://robotino_roller/description/mesh/roller01.stl
- link roller_leftupback_wheel0_link: geometry collision mesh filename=package://robotino_roller/description/mesh/roller01.stl; visual mesh filename=package://robotino_roller/description/mesh/roller01.stl
- link roller_leftupback_wheel1_link: geometry collision mesh filename=package://robotino_roller/description/mesh/roller01.stl; visual mesh filename=package://robotino_roller/description/mesh/roller01.stl
- link roller_leftupback_wheel2_link: geometry collision mesh filename=package://robotino_roller/description/mesh/roller01.stl; visual mesh filename=package://robotino_roller/description/mesh/roller01.stl
- link roller_leftupfront_wheel0_link: geometry collision mesh filename=package://robotino_roller/description/mesh/roller01.stl; visual mesh filename=package://robotino_roller/description/mesh/roller01.stl
- link roller_leftupfront_wheel1_link: geometry collision mesh filename=package://robotino_roller/description/mesh/roller01.stl; visual mesh filename=package://robotino_roller/description/mesh/roller01.stl
- link roller_leftupfront_wheel2_link: geometry collision mesh filename=package://robotino_roller/description/mesh/roller01.stl; visual mesh filename=package://robotino_roller/description/mesh/roller01.stl
- link roller_rightdownback_wheel0_link: geometry collision mesh filename=package://robotino_roller/description/mesh/roller01.stl; visual mesh filename=package://robotino_roller/description/mesh/roller01.stl
- link roller_rightdownback_wheel1_link: geometry collision mesh filename=package://robotino_roller/description/mesh/roller01.stl; visual mesh filename=package://robotino_roller/description/mesh/roller01.stl
- link roller_rightdownback_wheel2_link: geometry collision mesh filename=package://robotino_roller/description/mesh/roller01.stl; visual mesh filename=package://robotino_roller/description/mesh/roller01.stl
- link roller_rightdownfront_wheel0_link: geometry collision mesh filename=package://robotino_roller/description/mesh/roller01.stl; visual mesh filename=package://robotino_roller/description/mesh/roller01.stl
- link roller_rightdownfront_wheel1_link: geometry collision mesh filename=package://robotino_roller/description/mesh/roller01.stl; visual mesh filename=package://robotino_roller/description/mesh/roller01.stl
- link roller_rightdownfront_wheel2_link: geometry collision mesh filename=package://robotino_roller/description/mesh/roller01.stl; visual mesh filename=package://robotino_roller/description/mesh/roller01.stl
- link roller_rightupback_wheel0_link: geometry collision mesh filename=package://robotino_roller/description/mesh/roller01.stl; visual mesh filename=package://robotino_roller/description/mesh/roller01.stl
- link roller_rightupback_wheel1_link: geometry collision mesh filename=package://robotino_roller/description/mesh/roller01.stl; visual mesh filename=package://robotino_roller/description/mesh/roller01.stl
- link roller_rightupback_wheel2_link: geometry collision mesh filename=package://robotino_roller/description/mesh/roller01.stl; visual mesh filename=package://robotino_roller/description/mesh/roller01.stl
- link roller_rightupfront_wheel0_link: geometry collision mesh filename=package://robotino_roller/description/mesh/roller01.stl; visual mesh filename=package://robotino_roller/description/mesh/roller01.stl
- link roller_rightupfront_wheel1_link: geometry collision mesh filename=package://robotino_roller/description/mesh/roller01.stl; visual mesh filename=package://robotino_roller/description/mesh/roller01.stl
- link roller_rightupfront_wheel2_link: geometry collision mesh filename=package://robotino_roller/description/mesh/roller01.stl; visual mesh filename=package://robotino_roller/description/mesh/roller01.stl
- link roller_upback_wheel0_link: geometry collision mesh filename=package://robotino_roller/description/mesh/roller01.stl; visual mesh filename=package://robotino_roller/description/mesh/roller01.stl
- link roller_upback_wheel1_link: geometry collision mesh filename=package://robotino_roller/description/mesh/roller01.stl; visual mesh filename=package://robotino_roller/description/mesh/roller01.stl
- link roller_upback_wheel2_link: geometry collision mesh filename=package://robotino_roller/description/mesh/roller01.stl; visual mesh filename=package://robotino_roller/description/mesh/roller01.stl
- link roller_upfront_wheel0_link: geometry collision mesh filename=package://robotino_roller/description/mesh/roller01.stl; visual mesh filename=package://robotino_roller/description/mesh/roller01.stl
- link roller_upfront_wheel1_link: geometry collision mesh filename=package://robotino_roller/description/mesh/roller01.stl; visual mesh filename=package://robotino_roller/description/mesh/roller01.stl
- link roller_upfront_wheel2_link: geometry collision mesh filename=package://robotino_roller/description/mesh/roller01.stl; visual mesh filename=package://robotino_roller/description/mesh/roller01.stl
- link wheel0_link: geometry collision mesh filename=package://robotino_roller/description/mesh/rim01.stl; visual mesh filename=package://robotino_roller/description/mesh/rim01.stl
- link wheel1_link: geometry collision mesh filename=package://robotino_roller/description/mesh/rim01.stl; visual mesh filename=package://robotino_roller/description/mesh/rim01.stl
- link wheel2_link: geometry collision mesh filename=package://robotino_roller/description/mesh/rim01.stl; visual mesh filename=package://robotino_roller/description/mesh/rim01.stl

File: description/urdf/robotino.urdf.xacro (robot description, xacro)
@@ -15,9 +15,9 @@
         </xacro:inertial_cylinder>
         <visual>
-            <origin xyz="0 0 ${BASE_HEIGHT}" rpy="0 0 0" />
+            <!-- <origin xyz="0 0 ${BASE_HEIGHT}" rpy="0 0 0" /> -->
             <origin xyz="0.01 0 0" rpy="0 0 ${M_PI/2}"/>
             <geometry>
-                <cylinder radius="${BASE_RADIUS}" length="${BASE_HEIGHT}"/>
-                <mesh filename="package://robotino_sim/description/meshes/robotino_base.dae" scale="${M_SCALE} ${M_SCALE} ${M_SCALE}"/>
+                <!-- <cylinder radius="${BASE_RADIUS}" length="${BASE_HEIGHT}"/> -->
+                <mesh filename="package://robotino_roller/description/mesh/robotino_base.dae" scale="${M_SCALE} ${M_SCALE} ${M_SCALE}"/>
             </geometry>
         </visual>
@@ -50,55 +50,4 @@
         <axis xyz="0 0 1"/>
     </xacro:wheel_macro>
-    <!-- <xacro:macro name="wheel" params="parent name *origin *axis">
-        <link name="${name}_link">
-            <xacro:inertial_cylinder mass="${WHEEL_MASS}" height="${WHEEL_HEIGHT}" radius="${WHEEL_RADIUS}">
-                <origin xyz="0 0 0"/>
-            </xacro:inertial_cylinder>
-            <visual>
-                <origin xyz="0 0 0" rpy="0 0 0"/>
-                <geometry>
-                    <mesh filename="package://robotino_sim/description/meshes/robotino_wheel.dae" scale="${M_SCALE} ${M_SCALE} ${M_SCALE}"/>
-                </geometry>
-            </visual>
-            <collision>
-                <origin xyz="0 0 0" rpy="0 0 0"/>
-                <geometry>
-                    <mesh filename="package://robotino_sim/description/meshes/robotino_wheel.dae" scale="${M_SCALE} ${M_SCALE} ${M_SCALE}"/>
-                </geometry>
-            </collision>
-        </link>
-        <gazebo reference="${name}_link">
-            <material>Gazebo/Yellow</material>
-            <turnGravityOff>false</turnGravityOff>
-        </gazebo>
-        <joint name="${name}_joint" type="continuous">
-            <xacro:insert_block name="origin" />
-            <xacro:insert_block name="axis"/>
-            <parent link="${parent}"/>
-            <child link="${name}_link"/>
-        </joint>
-        <transmission name="${name}_joint_trans">
-            <type>transmission_interface/SimpleTransmission</type>
-            <joint name="${name}_joint">
-                <hardwareInterface>hardware_interface/EffortJointInterface</hardwareInterface>
-            </joint>
-            <actuator name="${name}_motor">
-                <hardwareInterface>hardware_interface/EffortJointInterface</hardwareInterface>
-                <mechanicalReduction>1</mechanicalReduction>
-            </actuator>
-        </transmission>
-    </xacro:macro>
-    <xacro:wheel name="wheel0o" parent="base_link">
-        <origin xyz="0.065 0.11 0.08" rpy="0 ${M_PI/2} ${M_PI/3}"/>
-        <axis xyz="-1 0 0"/>
-    </xacro:wheel>
-    <xacro:wheel name="wheel1o" parent="base_link">
-        <origin xyz="-0.13 0 0.08" rpy="0 ${M_PI/2} 0"/>
-        <axis xyz="1 0 0"/>
-    </xacro:wheel>
-    <xacro:wheel name="wheel2o" parent="base_link">
-        <origin xyz="0.065 -0.11 0.08" rpy="0 ${M_PI/2} -${M_PI/3}"/>
-        <axis xyz="-1 0 0"/>
-    </xacro:wheel> -->
     <gazebo>
         <plugin filename="libgazebo_ros_control.so" name="gazebo_ros_control"/>

File: description/urdf/wheel.xacro (robot description, xacro)
@@ -8,10 +8,12 @@
 			<visual>
 				<geometry>
-					<mesh filename="package://robotino_roller/description/mesh/rim.stl" scale="${M_SCALE} ${M_SCALE} ${M_SCALE}"/>
+					<mesh filename="package://robotino_roller/description/mesh/rim01.stl"/>
+					<!-- <mesh filename="package://robotino_roller/description/mesh/roda.stl" scale="${WHEEL_SCALE} ${WHEEL_SCALE} ${WHEEL_SCALE}"/> -->
 				</geometry>
 			</visual>
 			<collision>
 				<geometry>
-					<mesh filename="package://robotino_roller/description/mesh/rim.stl" scale="${M_SCALE} ${M_SCALE} ${M_SCALE}"/>
+					<mesh filename="package://robotino_roller/description/mesh/rim01.stl"/>
+					<!-- <mesh filename="package://robotino_roller/description/mesh/roda.stl" scale="${WHEEL_SCALE} ${WHEEL_SCALE} ${WHEEL_SCALE}"/> -->
 				</geometry>
 			</collision>
@@ -52,19 +54,17 @@
 	<xacro:macro name="roller_macro" params="parent name xyz rpy">
 		<link name="roller_${name}_${parent}_link">
-			<!-- <inertial>
-				<mass value="0.001"/>
-				<inertia ixx="3.976186554728152e-08" ixy="0" ixz="0" iyy="3.976186554728152e-08" iyz="0" izz="2.092071223656384e-08"/>
-			</inertial> -->
 			<xacro:inertial_cylinder mass="${ROLLER_MASS}" height="${ROLLER_HEIGHT*WHEEL_SCALE}" radius="${ROLLER_RADIUS*WHEEL_SCALE}">
-				<origin xyz="0 0 ${-0.000343*WHEEL_SCALE}"/>
+				<origin xyz="0 0 0"/>
 			</xacro:inertial_cylinder>
 			<visual>
 				<geometry>
-					<mesh filename="package://robotino_roller/description/mesh/roller.stl" scale="${M_SCALE} ${M_SCALE} ${M_SCALE}"/>
+					<mesh filename="package://robotino_roller/description/mesh/roller01.stl"/>
+					<!-- <mesh filename="package://robotino_roller/description/mesh/rolamento.stl" scale="${WHEEL_SCALE} ${WHEEL_SCALE} ${WHEEL_SCALE}"/> -->
 				</geometry>
 			</visual>
 			<collision>
 				<geometry>
-					<mesh filename="package://robotino_roller/description/mesh/roller.stl" scale="${M_SCALE} ${M_SCALE} ${M_SCALE}"/>
+					<mesh filename="package://robotino_roller/description/mesh/roller01.stl"/>
+					<!-- <mesh filename="package://robotino_roller/description/mesh/rolamento.stl" scale="${WHEEL_SCALE} ${WHEEL_SCALE} ${WHEEL_SCALE}"/> -->
 				</geometry>
 			</collision>
@@ -72,8 +72,8 @@
 		<gazebo reference="roller_${name}_${parent}_link">
 			<material>Gazebo/Black</material>
-			<!-- <mu1 value="2.5" />
+			<mu1 value="2.5" />
 			<mu2 value="2.5" />
 			<kp value="5000" />
-			<kd value="10" /> -->
+			<kd value="10" />
 		</gazebo>
 		<joint name="roller_${name}_${parent}_joint" type="continuous">
